File: microphone-board.kicad_pcb (KiCad board)
At the start: 4 copper layers, 10.7 x 11 mm, 13 parts, among them J1 Conn_FFC_Molex_5019510550

Commit message: [#71249] Update name
Other:
- board text added: "Microphone Board Rev. ${REVISION}"
- board text removed: "Audio Microphone Rev. ${REVISION}"
Changed lines of the file:
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@@
 	(paper "A3")
 	(title_block
-		(title "Audio Microphone")
+		(title "Microphone board")
 		(date "2025-01-24")
 		(rev "1.2.0")
@@
 		)
 		(sheetname "Root")
-		(sheetfile "microphone-pcb.kicad_sch")
+		(sheetfile "microphone-board.kicad_sch")
 		(attr smd)
 		(fp_rect
@@
 		)
 		(sheetname "Root")
-		(sheetfile "microphone-pcb.kicad_sch")
+		(sheetfile "microphone-board.kicad_sch")
 		(attr smd)
 		(fp_rect
@@
 		)
 		(sheetname "Root")
-		(sheetfile "microphone-pcb.kicad_sch")
+		(sheetfile "microphone-board.kicad_sch")
 		(attr smd)
 		(fp_rect
@@
 		)
 		(sheetname "Root")
-		(sheetfile "microphone-pcb.kicad_sch")
+		(sheetfile "microphone-board.kicad_sch")
 		(attr smd)
 		(fp_rect
@@
 		)
 		(sheetname "Root")
-		(sheetfile "microphone-pcb.kicad_sch")
+		(sheetfile "microphone-board.kicad_sch")
 		(attr smd)
 		(fp_rect
@@
 		)
 		(sheetname "Root")
-		(sheetfile "microphone-pcb.kicad_sch")
+		(sheetfile "microphone-board.kicad_sch")
 		(attr smd)
 		(fp_rect
@@
 		)
 		(sheetname "Root")
-		(sheetfile "microphone-pcb.kicad_sch")
+		(sheetfile "microphone-board.kicad_sch")
 		(attr smd exclude_from_pos_files exclude_from_bom dnp)
 		(fp_poly
@@
 		)
 		(sheetname "Root")
-		(sheetfile "microphone-pcb.kicad_sch")
+		(sheetfile "microphone-board.kicad_sch")
 		(attr smd)
 		(fp_line
@@
 		)
 		(sheetname "Root")
-		(sheetfile "microphone-pcb.kicad_sch")
+		(sheetfile "microphone-board.kicad_sch")
 		(attr smd)
 		(fp_poly
@@
 		)
 		(sheetname "Root")
-		(sheetfile "microphone-pcb.kicad_sch")
+		(sheetfile "microphone-board.kicad_sch")
 		(attr smd)
 		(fp_rect
@@
 		)
 		(sheetname "Root")
-		(sheetfile "microphone-pcb.kicad_sch")
+		(sheetfile "microphone-board.kicad_sch")
 		(attr smd)
 		(fp_poly
@@
 		)
 		(sheetname "Root")
-		(sheetfile "microphone-pcb.kicad_sch")
+		(sheetfile "microphone-board.kicad_sch")
 		(attr smd)
 		(fp_rect
@@
 		)
 		(sheetname "Root")
-		(sheetfile "microphone-pcb.kicad_sch")
+		(sheetfile "microphone-board.kicad_sch")
 		(attr smd)
 		(fp_poly
@@
 		(layer "Edge.Cuts")
 	)
-	(gr_text "Audio\nMicrophone\nRev. ${REVISION}"
+	(gr_text "Microphone\nBoard\nRev. ${REVISION}"
 		(at 239.9462 151.5266 0)
 		(layer "B.SilkS")
