File: microphone-board.kicad_pcb (KiCad board)
At the start: 4 copper layers, 10.7 x 11 mm, 12 parts, among them J1 Conn_FFC_Molex_5019510550

Commit message: [#75547] Add license and logotype
Parts:
- added REF**: OSHW-Logo_5.7x6mm_SilkScreen, antmicro-footprints:OSHW-Logo_5.7x6mm_SilkScreen, B.Cu at (240.0, 144.9)
Other:
- board text added: "SHA:######## PDM Mic. Board Rev.${REVISION}"
- board text removed: "Microphone Board Rev. ${REVISION}"
- board text removed: "SHA:########"
